Commit message: Added depth camera

File: src/robotic_arm_description/urdf/camera.xacro (robot description, xacro)
@@ -16,8 +16,8 @@
         </collision>
         <xacro:box_inertia m="0.1" x="0.1" y="0.1" z="0.05"
-                           o_xyz="0 0 0" o_rpy="0 0 0"/>
+            o_xyz="0 0 0" o_rpy="0 0 0"/>
     </link>
     <link name="virtual_camera"/>
-    <joint name="camera_link_optical" type="fixed" >
+    <joint name="camera_link_optical" type="fixed">
         <parent link="camera_link"/>
         <child link="virtual_camera"/>
@@ -25,5 +25,5 @@
     </joint>
     <gazebo reference="camera_link">
-        <sensor name="camera" type="camera">
+        <sensor name="depth_camera" type="rgbd_camera">
             <camera>
                 <horizontal_fov>1.3962634</horizontal_fov>
@@ -48,5 +48,5 @@
             <update_rate>20</update_rate>
             <visualize>true</visualize>
-            <topic>camera/image_raw</topic>
+            <topic>camera</topic>
         </sensor>
     </gazebo>
